File: kicad/sneksafe.kicad_pcb (KiCad board)
At the start: 2 copper layers, 143 x 78 mm, 15 parts, among them J1 BME280, J2 Screw_Terminal_01x06, J3 Screw_Terminal_01x03, K1 CPC40055ST, K2 CPC40055ST, U1 ESP32-DEVKITC-32D

Commit message: board v1.1: add mounting holes and update QR link
Parts:
- moved QR***** 11.9 mm to (211.8, 80.2)
Routing:
- net Earth: vias 0 -> 2
- net (no net): vias 0 -> 2
Other:
- board text added: "SnekSafe v1.1"
- board text removed: "SnekSafe v1.0"

Commit message: pcb: prepare for CI-generated BOM
Parts:
- J1: value BME280 -> S4B-XH-A(LF)(SN)
Changed lines of the file:
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@@
     (descr "Resistor SMD 1206 (3216 Metric), square (rectangular) end terminal, IPC_7351 nominal with elongated pad for handsoldering. (Body size source: IPC-SM-782 page 72, https://www.pcb-3d.com/wordpress/wp-content/uploads/ipc-sm-782a_amendment_1_and_2.pdf), generated with kicad-footprint-generator")
     (tags "resistor handsolder")
+    (property "Manufacturer_Name" "Panasonic")
+    (property "Manufacturer_Part_Number" "ERA-8AEB242V")
+    (property "Price" "$0.64")
+    (property "Product Link" "https://www.mouser.com/ProductDetail/667-ERA-8AEB242V")
     (property "Sheetfile" "sneksafe.kicad_sch")
     (property "Sheetname" "")
@@
     (descr "Resistor SMD 1206 (3216 Metric), square (rectangular) end terminal, IPC_7351 nominal with elongated pad for handsoldering. (Body size source: IPC-SM-782 page 72, https://www.pcb-3d.com/wordpress/wp-content/uploads/ipc-sm-782a_amendment_1_and_2.pdf), generated with kicad-footprint-generator")
     (tags "resistor handsolder")
+    (property "Manufacturer_Name" "Panasonic")
+    (property "Manufacturer_Part_Number" "ERA-8AEB242V")
+    (property "Price" "$0.64")
+    (property "Product Link" "https://www.mouser.com/ProductDetail/667-ERA-8AEB242V")
     (property "Sheetfile" "sneksafe.kicad_sch")
     (property "Sheetname" "")
@@
     (property "MANUFACTURER" "Espressif Systems")
     (property "MAXIMUM_PACKAGE_HEIGHT" "N/A")
+    (property "Manufacturer_Name" "Espressif Systems ")
+    (property "Manufacturer_Part_Number" "ESP32-DevKitC-32E")
     (property "PARTREV" "V4")
+    (property "Price" "$10.00")
+    (property "Product Link" "https://www.mouser.com/ProductDetail/356-ESP32-DEVKITC32E")
     (property "SNAPEDA_PN" "ESP32-DEVKITC-32D")
     (property "STANDARD" "Manufacturer Recommendations")
@@
     (descr "Resistor SMD 1206 (3216 Metric), square (rectangular) end terminal, IPC_7351 nominal with elongated pad for handsoldering. (Body size source: IPC-SM-782 page 72, https://www.pcb-3d.com/wordpress/wp-content/uploads/ipc-sm-782a_amendment_1_and_2.pdf), generated with kicad-footprint-generator")
     (tags "resistor handsolder")
+    (property "Manufacturer_Name" "Panasonic")
+    (property "Manufacturer_Part_Number" "ERA-8AEB103V")
+    (property "Price" "$0.70")
+    (property "Product Link" "https://www.mouser.com/ProductDetail/667-ERA-8AEB103V")
     (property "Sheetfile" "sneksafe.kicad_sch")
     (property "Sheetname" "")
@@
     (descr "Resistor SMD 1206 (3216 Metric), square (rectangular) end terminal, IPC_7351 nominal with elongated pad for handsoldering. (Body size source: IPC-SM-782 page 72, https://www.pcb-3d.com/wordpress/wp-content/uploads/ipc-sm-782a_amendment_1_and_2.pdf), generated with kicad-footprint-generator")
     (tags "resistor handsolder")
+    (property "Manufacturer_Name" "Panasonic")
+    (property "Manufacturer_Part_Number" "ERA-8AEB4220V")
+    (property "Price" "$0.66")
+    (property "Product Link" "https://www.mouser.com/ProductDetail/667-ERA-8AEB4220V")
     (property "Sheetfile" "sneksafe.kicad_sch")
     (property "Sheetname" "")
@@
     (descr "1713969-2")
     (tags "Connector")
+    (property "Manufacturer_Name" "Phoenix Contact ")
+    (property "Manufacturer_Part_Number" "1713969")
+    (property "Price" "$5.84")
+    (property "Product Link" "https://www.mouser.com/ProductDetail/651-1713969")
     (property "Sheetfile" "sneksafe.kicad_sch")
     (property "Sheetname" "")
@@
     (property "Mouser Part Number" "919-RAC10E-05SK/277")
     (property "Mouser Price/Stock" "https://www.mouser.co.uk/ProductDetail/RECOM-Power/RAC10E-05SK-277?qs=Li%252BoUPsLEnvJW5q%2F0CCh4A%3D%3D")
+    (property "Price" "$9.55")
+    (property "Product Link" "https://www.mouser.com/ProductDetail/919-RAC10E-05SK-277")
     (property "Sheetfile" "sneksafe.kicad_sch")
     (property "Sheetname" "")
@@
     (descr "Resistor SMD 1206 (3216 Metric), square (rectangular) end terminal, IPC_7351 nominal with elongated pad for handsoldering. (Body size source: IPC-SM-782 page 72, https://www.pcb-3d.com/wordpress/wp-content/uploads/ipc-sm-782a_amendment_1_and_2.pdf), generated with kicad-footprint-generator")
     (tags "resistor handsolder")
+    (property "Manufacturer_Name" "Panasonic")
+    (property "Manufacturer_Part_Number" "ERA-8AEB4220V")
+    (property "Price" "$0.66")
+    (property "Product Link" "https://www.mouser.com/ProductDetail/667-ERA-8AEB4220V")
     (property "Sheetfile" "sneksafe.kicad_sch")
     (property "Sheetname" "")
@@
     (descr "JST XH series connector, S4B-XH-A (http://www.jst-mfg.com/product/pdf/eng/eXH.pdf), generated with kicad-footprint-generator")
     (tags "connector JST XH horizontal")
+    (property "Manufacturer_Name" "JST")
+    (property "Manufacturer_Part_Number" "S4B-XH-A(LF)(SN)")
+    (property "Price" "$0.27")
+    (property "Product Link" "https://www.digikey.com/en/products/detail/jst-sales-america-inc/S4B-XH-A-LF-SN/1651041")
     (property "Sheetfile" "sneksafe.kicad_sch")
     (property "Sheetname" "")
@@
         (effects (font (size 1 1) (thickness 0.15)))
     )
-    (fp_text value "BME280" (at -5.75 0.85) (layer "F.Fab")
+    (fp_text value "S4B-XH-A(LF)(SN)" (at -5.75 0.85) (layer "F.Fab")
         (effects (font (size 1 1) (thickness 0.15)))
     )
@@
     (tags "Relay or Contactor")
     (property "Height" "20.701")
-    (property "Manufacturer_Name" "LITTELFUSE")
+    (property "Manufacturer_Name" "Littelfuse")
     (property "Manufacturer_Part_Number" "CPC40055ST")
     (property "Mouser Part Number" "849-CPC40055ST")
     (property "Mouser Price/Stock" "https://www.mouser.co.uk/ProductDetail/IXYS-Integrated-Circuits/CPC40055ST?qs=%2FWJw0caR6035dTiWeJluMw%3D%3D")
+    (property "Price" "$13.35")
+    (property "Product Link" "https://www.mouser.com/ProductDetail/849-CPC40055ST")
     (property "Sheetfile" "sneksafe.kicad_sch")
     (property "Sheetname" "")
@@
     (descr "Capacitor SMD 1206 (3216 Metric), square (rectangular) end terminal, IPC_7351 nominal with elongated pad for handsoldering. (Body size source: IPC-SM-782 page 76, https://www.pcb-3d.com/wordpress/wp-content/uploads/ipc-sm-782a_amendment_1_and_2.pdf), generated with kicad-footprint-generator")
     (tags "capacitor handsolder")
+    (property "Manufacturer_Name" "Murata")
+    (property "Manufacturer_Part_Number" "GRM31CR72A105KA01K")
+    (property "Price" "$0.78")
+    (property "Product Link" "https://www.mouser.com/ProductDetail/81-GRM31CR72A105KA1K")
     (property "Sheetfile" "sneksafe.kicad_sch")
     (property "Sheetname" "")
@@
     (descr "1714968-2")
     (tags "Connector")
+    (property "Manufacturer_Name" "Phoenix Contact ")
+    (property "Manufacturer_Part_Number" "1714968")
+    (property "Price" "$2.79")
+    (property "Product Link" "https://www.mouser.com/ProductDetail/651-1714968")
     (property "Sheetfile" "sneksafe.kicad_sch")
     (property "Sheetname" "")
@@
     (tags "Relay or Contactor")
     (property "Height" "20.701")
-    (property "Manufacturer_Name" "LITTELFUSE")
+    (property "Manufacturer_Name" "Littelfuse")
     (property "Manufacturer_Part_Number" "CPC40055ST")
     (property "Mouser Part Number" "849-CPC40055ST")
     (property "Mouser Price/Stock" "https://www.mouser.co.uk/ProductDetail/IXYS-Integrated-Circuits/CPC40055ST?qs=%2FWJw0caR6035dTiWeJluMw%3D%3D")
+    (property "Price" "$13.35")
+    (property "Product Link" "https://www.mouser.com/ProductDetail/849-CPC40055ST")
     (property "Sheetfile" "sneksafe.kicad_sch")
     (property "Sheetname" "")

Commit message: Prepare for kibot
Parts:
- added MH1: MountingHole_3.2mm_M3_Pad_Via, MountingHole:MountingHole_3.2mm_M3_Pad_Via, F.Cu at (161.8, 83.2)
- added MH2: MountingHole_3.2mm_M3_Pad_Via, MountingHole:MountingHole_3.2mm_M3_Pad_Via, F.Cu at (217.2, 96.0)
- added MH3: MountingHole_Pad, MountingHole:MountingHole_3.2mm_M3_Pad_Via, F.Cu at (135.0, 139.2)
- added MH4: MountingHole_Pad, MountingHole:MountingHole_3.2mm_M3_Pad_Via, F.Cu at (186.8, 119.8)
Connections:
- J2 pad 3: Earth -> Net-(J2-Pin_3)
- J2 pad 6: Earth -> Net-(J2-Pin_6)
- J3 pad 2: Earth -> Net-(J3-Pin_2)
Routing:
- net Earth: vias 2 -> 0
- net (no net): vias 2 -> 0
