File: kicad/sneksafe.kicad_pcb (KiCad board)
At the start: 2 copper layers, 143 x 78 mm, 19 parts, among them J1 S4B-XH-A(LF)(SN), J2 Screw_Terminal_01x06, J3 Screw_Terminal_01x03, K1 CPC40055ST, K2 CPC40055ST, U1 ESP32-DEVKITC-32D

Commit message: board v1.2
Parts:
- removed G***: LOGO, snek:snek
- added U2: DS1307+, Package_DIP:DIP-8_W7.62mm, F.Cu at (170.2, 85.9)
- added U3: 1074, Keystone 1074:1074, F.Cu at (181.4, 70.1)
- added Y1: 830003000, 830003000:830003000, F.Cu at (179.0, 83.2)
- moved MH1 12.8 mm to (166.2, 71.2)
- moved QR***** 1.86 mm to (213.4, 79.4)
Routing:
- net AC_P_IN: track 0.00 -> 289.1 mm, vias 0 -> 26
- net AC_N_IN: track 108.1 -> 351.5 mm, vias 0 -> 27
- net LIGHT_AC_P: track 43.8 -> 89.6 mm, vias 0 -> 9
- net Net-(U2-VBAT): track 0.00 -> 25.6 mm
- net HEAT_AC_P: track 19.4 -> 39.4 mm, vias 0 -> 3
- net SCL: track 42.2 -> 57.6 mm
- net SDA: track 53.8 -> 65.8 mm
- net +5V: track 99.0 -> 108.7 mm
- net Net-(U2-X1): track 0.00 -> 6.69 mm
- net Net-(U2-X2): track 0.00 -> 6.59 mm
- removed copper zone on F.Cu, net AC_N_IN
- removed copper zone on F.Cu, net AC_P_IN
Other:
- board size 143 x 78 mm -> 143.2 x 81.4 mm
- board text added: "Copyright © 2018-2024 Jacob McSwain"
- board text added: "SnekSafe v1.2"
- board text removed: "Copyright © 2018-2023 Jacob McSwain"
- board text removed: "SnekSafe v1.1"
