File: kicad/sneksafe.kicad_sch (KiCad schematic)
At the start: 26 parts, among them J1 S4B-XH-A(LF)(SN), J2 Screw_Terminal_01x06, J3 Screw_Terminal_01x03, K1 CPC40055ST, K2 CPC40055ST, U1 ESP32-DEVKITC-32D

Commit message: Prepare for kibot
Parts:
- added MH3, MH4: MountingHole_Pad, MountingHole:MountingHole_3.2mm_M3_Pad_Via, symbol Mechanical:MountingHole_Pad
- ACCord1: Manufacturer_Name Cable Leader -> CableLeader
- J2, J3: Manufacturer_Name Phoenix Contact -> PhoenixContact
- PS1: footprint RAC10E-05SK_277:RAC10E05SK277 -> RAC10E05SK277; Manufacturer_Name RECOM Power -> RECOMPower
- U1: Manufacturer_Name Espressif Systems -> EspressifSystems
Connections:
- net Earth: now also MH3.1, MH4.1; no longer J2.3 (Pin_3), J2.6 (Pin_6), J3.2 (Pin_2)
- no-connect marks 28 -> 54
Other:
- moved on the sheet: HS1, HS2

Commit message: kicad: fixups
Parts:
- ACCord1: Amazon Link (none) -> https://www.amazon.com/dp/B07KBDPH8X; Manufacturer_Name CableLeader -> Cable Leader; Product Link https://www.amazon.com/dp/B07KBDPH8X -> (none)
- ACFuse1: Digikey Link (none) -> https://www.digikey.com/en/products/detail/littelfuse-inc/0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; Mouser Link (none) -> https://www.mouser.com/ProductDetail/576-0215010.MXF60P; Product Link https://www.mouser.com/ProductDetail/576-0215010.MXF60P -> (none)
- ACOutput1, ACOutput2: Amazon Link (none) -> https://www.amazon.com/dp/B09V27W6H6; Product Link https://www.amazon.com/dp/B09V27W6H6 -> (none)
- ACPlug1: Amazon Link (none) -> https://www.amazon.com/dp/B0895T9NXF; Product Link https://www.amazon.com/dp/B0895T9NXF -> (none)
- C1: Digikey Link (none) -> https://www.digikey.com/en/products/detail/murata-electroni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; Mouser Link (none) -> https://www.mouser.com/ProductDetail/81-GRM31CR72A105KA1K; Product Link https://www.mouser.com/ProductDetail/81-GRM31CR72A105KA1K -> (none)
- HS1, HS2: Digikey Link (none) -> https://www.digikey.com/en/products/detail/aavid-thermal-di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; Mouser Link (none) -> https://www.mouser.com/ProductDetail/532-508500B00; Product Link https://www.mouser.com/ProductDetail/532-508500B00 -> (none)
- J1, TempPlug1, TempPlugCrimp1, TempPlugCrimp2, TempPlugCrimp3, TempPlugCrimp4: Digikey Link (none) -> https://www.digikey.com/en/products/detail/jst-sales-americ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; Product Link https://www.digikey.com/en/products/detail/jst-sales-americ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 -> (none)
- J2: Digikey Link (none) -> https://www.digikey.com/en/products/detail/phoenix-contact/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; Manufacturer_Name PhoenixContact -> Phoenix Contact; Mouser Link (none) -> https://www.mouser.com/ProductDetail/651-1713969; Product Link https://www.mouser.com/ProductDetail/651-1713969 -> (none)
- J3: Digikey Link (none) -> https://www.digikey.com/en/products/detail/phoenix-contact/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; Manufacturer_Name PhoenixContact -> Phoenix Contact; Mouser Link (none) -> https://www.mouser.com/ProductDetail/651-1714968; Product Link https://www.mouser.com/ProductDetail/651-1714968 -> (none)
- K1, K2: Digikey Link (none) -> https://www.digikey.com/en/products/detail/ixys-integrated-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; Height 20.701 -> (none); Manufacturer_Name Littelfuse -> IXYS Integrated Circuits Division; Mouser Link (none) -> https://www.mouser.com/ProductDetail/849-CPC40055ST; Mouser Part Number 849-CPC40055ST -> (none); Mouser Price/Stock https://www.mouser.co.uk/ProductDetail/IXYS-Integrated-Circ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 -> (none); Product Link https://www.mouser.com/ProductDetail/849-CPC40055ST -> (none)
- MH3, MH4: now left out of the parts list
- PS1: Digikey Link (none) -> https://www.digikey.com/en/products/detail/recom-power/RAC1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; Height 22 -> (none); Manufacturer_Name RECOMPower -> RECOM Power; Mouser Link (none) -> https://www.mouser.com/ProductDetail/919-RAC10E-05SK-277; Mouser Part Number 919-RAC10E-05SK/277 -> (none); Mouser Price/Stock https://www.mouser.co.uk/ProductDetail/RECOM-Power/RAC10E-0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 -> (none); Product Link https://www.mouser.com/ProductDetail/919-RAC10E-05SK-277 -> (none)
- R1, R2: Digikey Link (none) -> https://www.digikey.com/en/products/detail/panasonic-electr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; Mouser Link (none) -> https://www.mouser.com/ProductDetail/667-ERA-8AEB242V; Product Link https://www.mouser.com/ProductDetail/667-ERA-8AEB242V -> (none)
- R3: Digikey Link (none) -> https://www.digikey.com/en/products/detail/panasonic-electr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; Mouser Link (none) -> https://www.mouser.com/ProductDetail/667-ERA-8AEB103V; Product Link https://www.mouser.com/ProductDetail/667-ERA-8AEB103V -> (none)
- R5, R6: Digikey Link (none) -> https://www.digikey.com/en/products/detail/panasonic-electr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; Mouser Link (none) -> https://www.mouser.com/ProductDetail/667-ERA-8AEB4220V; Product Link https://www.mouser.com/ProductDetail/667-ERA-8AEB4220V -> (none)
- TempSensor1: Digikey Link (none) -> https://www.digikey.com/en/products/detail/dfrobot/SEN0385/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; Mouser Link (none) -> https://www.mouser.com/ProductDetail/426-SEN0385; Product Link https://www.mouser.com/ProductDetail/426-SEN0385 -> (none)
- U1: Digikey Link (none) -> https://www.digikey.com/en/products/detail/espressif-system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; MANUFACTURER Espressif Systems -> (none); MAXIMUM_PACKAGE_HEIGHT N/A -> (none); Manufacturer_Name EspressifSystems -> Espressif Systems; Mouser Link (none) -> https://www.mouser.com/ProductDetail/356-ESP32-DEVKITC32E; PARTREV V4 -> (none); Product Link https://www.mouser.com/ProductDetail/356-ESP32-DEVKITC32E -> (none); SNAPEDA_PN ESP32-DEVKITC-32D -> (none); STANDARD Manufacturer Recommendations -> (none)

Commit message: board v1.2
Parts:
- added U2: DS1307+, Package_DIP:DIP-8_W7.62mm, symbol Timer_RTC:DS1307+
- added U3: 1074, Keystone 1074:1074, symbol Keystone 1074:1074
- added Y1: 830003000, 830003000:830003000, symbol 830003000:830003000
- PS1: footprint RAC10E05SK277 -> RAC10E-05SK_277:RAC10E05SK277
Connections:
- net +5V: now also U2.8 (VCC)
- net GND: now also U2.4 (GND), U3.1, U3.2
- net SCL: now also U2.6 (SCL)
- net SDA: now also U2.5 (SDA)
- new net: U2.1 (X1), Y1.1 (CRYSTAL__1)
- new net: U2.2 (X2), Y1.4 (CRYSTAL__2)
- new net: U2.3 (VBAT), U3.3
- no-connect marks 54 -> 57
